File: New Panel/Isolinear Chip Board/Isolinear Board PCB/Isolinear Board PCB.kicad_pcb (KiCad board)
At the start: 2 copper layers, 58.2 x 32 mm, 23 parts, among them J1 Conn_01x02_Pin, J2 Conn_01x02_Pin, J3 Conn_01x02_Pin, J4 Conn_01x02_Pin, J5 Conn_01x02_Pin, J6 IN, J7 OUT, U1 74HC595

Commit message: Work on new main pcb
Parts:
- added C1: 10uF, Capacitor_THT:C_Disc_D5.0mm_W2.5mm_P5.00mm, B.Cu at (121.8, 139.2)
- added C2: 10uF, Capacitor_THT:C_Disc_D5.0mm_W2.5mm_P5.00mm, B.Cu at (136.2, 139.0)
- added JP4: SolderJumper_2_Bridged, Jumper:SolderJumper-2_P1.3mm_Bridged2Bar_RoundedPad1.0x1.5mm, B.Cu at (120.8, 142.0)
- added JP5: SolderJumper_2_Open, Jumper:SolderJumper-2_P1.3mm_Open_RoundedPad1.0x1.5mm, B.Cu at (120.8, 144.5)
- JP1, JP2, JP3: value SolderJumper_2_Open -> SolderJumper_2_Bridged; footprint Jumper:SolderJumper-2_P1.3mm_Open_TrianglePad1.0x1.5mm -> Jumper:SolderJumper-2_P1.3mm_Bridged2Bar_RoundedPad1.0x1.5mm
- moved JP2 3.50 mm to (120.0, 133.9)
- moved JP1 3.50 mm to (123.5, 134.0)
- moved JP3 0.10 mm to (116.5, 133.9), turned to -90 degrees
Connections:
- D1 pad 2: GND -> Net-(D1-GND)
- JP1 pad 1: Net-(D1-VDD) -> Net-(D1-DIN)
- JP1 pad 2: +5V -> /LED_DIN
- JP2 pad 1: Net-(D1-DIN) -> Net-(D1-VDD)
- JP2 pad 2: /LED_DIN -> +5V
- JP3 pad 1: Net-(D1-DOUT) -> /LED_Dout
- JP3 pad 2: /LED_Dout -> Net-(D1-DOUT)
Routing:
- net Net-(D1-GND): track 0.00 -> 6.59 mm
- net +5V: track 104.9 -> 109.2 mm
- net /LED_Dout: track 86.9 -> 82.9 mm
- net +3V3: track 65.4 -> 68.7 mm
- net /MCU_ANALOG: track 63.4 -> 62.0 mm
- net Net-(D1-VDD): track 10.6 -> 11.8 mm
- net /Switch 3: track 45.7 -> 45.0 mm
- net GND: vias 61 -> 82
Other:
- board text added: "Break J4 and bridge J5 for CMN VCC LED"
