File: New Panel/Isolinear Chip Board/Isolinear Board PCB/Isolinear Board PCB.kicad_sch (KiCad schematic)
At the start: 23 parts, among them J1 Conn_01x02_Pin, J2 Conn_01x02_Pin, J3 Conn_01x02_Pin, J4 Conn_01x02_Pin, J5 Conn_01x02_Pin, J6 IN, J7 OUT, U1 74HC595

Commit message: Work on new main pcb
Parts:
- removed JP1, JP2, JP3: SolderJumper_2_Open, Jumper:SolderJumper-2_P1.3mm_Open_TrianglePad1.0x1.5mm, symbol Jumper:SolderJumper_2_Open
- added C1, C2: 10uF, Capacitor_THT:C_Disc_D5.0mm_W2.5mm_P5.00mm, symbol Device:C
- added JP1, JP2, JP3, JP4: SolderJumper_2_Bridged, Jumper:SolderJumper-2_P1.3mm_Bridged2Bar_RoundedPad1.0x1.5mm, symbol Jumper:SolderJumper_2_Bridged
- added JP5: SolderJumper_2_Open, Jumper:SolderJumper-2_P1.3mm_Open_RoundedPad1.0x1.5mm, symbol Jumper:SolderJumper_2_Open
Connections:
- net +3V3: now also C2.1
- net +5V: now also JP2.2 (B), JP5.1 (A)
- net GND: now also C1.2, C2.2, JP4.2 (B); no longer D1.2 (GND)
- net LED_DIN: now also JP1.2 (B)
- net LED_Dout: now also JP3.1 (A)
- net at D1.3 (VDD), R3.2: now also C1.1, JP2.1 (A)
- net at D1.4 (DIN), R4.2: now also JP1.1 (A)
- net at D1.1 (DOUT), R2.2: now also JP3.2 (B)
- new net: D1.2 (GND), JP4.1 (A), JP5.2 (B)
