File: New Panel/Main Board/IO Expanders.kicad_sch (KiCad schematic)
At the start: 15 parts, among them J103 Conn_02x08_Odd_Even, J104 Conn_02x08_Odd_Even, J105 Conn_02x08_Odd_Even, J106 Conn_02x08_Odd_Even, J107 Conn_02x08_Odd_Even, J108 Conn_02x08_Odd_Even, J109 Conn_02x08_Odd_Even, U23 IO_EXPANDER_TCA9535PWR, U24 IO_EXPANDER_TCA9535PWR, U25 IO_EXPANDER_TCA9535PWR, U26 IO_EXPANDER_TCA9535PWR, U27 IO_EXPANDER_TCA9535PWR, U28 IO_EXPANDER_TCA9535PWR, U29 IO_EXPANDER_TCA9535PWR

Commit message: adjusted schematic and started PCB Work
Parts:
- removed J104, J105, J106, J107, J108, J109: Conn_02x08_Odd_Even, Connector_IDC:IDC-Header_2x08_P2.54mm_Vertical, symbol Connector_Generic:Conn_02x08_Odd_Even
- removed U24, U25, U26, U27, U28, U29: IO_EXPANDER_TCA9535PWR, New Panel Parts:24-TSSOP_(4.4mm), symbol New_Panel_Parts:IO_EXPANDER_TCA9535PWR
- added C13, C14, C15, C16, C17, C18, C19, C23, C24, C25, C26, C27, C28, C29, C30, C31, C32, C33, C34, C35, C36, C37, C38, C39, C40, C41, C42, C43, C44, C45, C46, C47, C48, C49, C50, C51, C52, C53, C54, C55, C56, C57, C58, C59, C60, C61, C62, C63, C64, C65, C66, C67, C68, C69, C70, C71, C72, C73, C74, C75, C76, C77, C78, C79: 0.1uF, Capacitor_SMD:C_0603_1608Metric_Pad1.08x0.95mm_HandSolder, symbol Device:C
- added D1, D10, D11, D12, D13, D14, D15, D16, D17, D18, D19, D2, D20, D21, D22, D23, D24, D25, D26, D27, D28, D29, D3, D30, D31, D32, D33, D34, D35, D36, D37, D38, D39, D4, D40, D41, D42, D43, D44, D45, D46, D47, D48, D49, D5, D50, D51, D52, D53, D54, D55, D56, D57, D58, D59, D6, D60, D61, D62, D63, D64, D7, D8, D9: DESD5V0S1BA-7, Diode_SMD:D_SOD-323, symbol Diode:SD05_SOD323
- added J46, J47, J48: Conn_02x08_Odd_Even, Connector_IDC:IDC-Header_2x08_P2.54mm_Vertical, symbol Connector_Generic:Conn_02x08_Odd_Even
- added R100, R103, R104, R107, R108, R111, R112, R115, R116, R119, R120, R123, R124, R127, R128, R165, R166, R167, R168, R173, R174, R175, R176, R181, R182, R183, R184, R189, R190, R191, R192, R197, R198, R199, R200, R205, R206, R207, R208, R213, R214, R215, R216, R221, R222, R223, R224, R67, R68, R69, R70, R71, R72, R73, R74, R83, R85, R87, R89, R91, R93, R95, R97, R99: 100K, Resistor_SMD:R_0603_1608Metric, symbol Device:R
- added R101, R102, R105, R106, R109, R110, R113, R114, R117, R118, R121, R122, R125, R126, R129, R163, R169, R170, R171, R172, R177, R178, R179, R180, R185, R186, R187, R188, R193, R194, R195, R196, R201, R202, R203, R204, R209, R210, R211, R212, R217, R218, R219, R220, R225, R226, R227, R228, R75, R76, R77, R78, R79, R80, R81, R82, R84, R86, R88, R90, R92, R94, R96, R98: 150R, Resistor_SMD:R_0603_1608Metric, symbol Device:R
- added TP21, TP22, TP23, TP24: TestPoint, Connector_Pin:Pin_D1.0mm_L10.0mm, symbol Connector:TestPoint
- added U11, U12, U13: IO_EXPANDER_TCA9535PWR, New Panel Parts:24-TSSOP_(4.4mm), symbol New_Panel_Parts:IO_EXPANDER_TCA9535PWR
- R158: now not fitted
Connections:
- net GND: now also C13.2, C14.2, C15.2, C16.2, C17.2, C18.2, C19.2, C23.2, C24.2, C25.2, C26.2, C27.2, C28.2, C29.2, C30.2, C31.2, C32.2, C33.2, C34.2, C35.2, C36.2, C37.2, C38.2, C39.2, C40.2, C41.2, C42.2, C43.2, C44.2, C45.2, C46.2, C47.2, C48.2, C49.2, C50.2, C51.2, C52.2, C53.2, C54.2, C55.2, C56.2, C57.2, C58.2, C59.2, C60.2, C61.2, C62.2, C63.2, C64.2, C65.2, C66.2, C67.2, C68.2, C69.2, C70.2, C71.2, C72.2, C73.2, C74.2, C75.2, C76.2, C77.2, C78.2, C79.2, D1.2 (A2), D10.2 (A2), D11.2 (A2), D12.2 (A2), D13.2 (A2), D14.2 (A2), D15.2 (A2), D16.2 (A2), D17.2 (A2), D18.2 (A2), D19.2 (A2), D2.2 (A2), D20.2 (A2), D21.2 (A2), D22.2 (A2), D23.2 (A2), D24.2 (A2), D25.2 (A2), D26.2 (A2), D27.2 (A2), D28.2 (A2), D29.2 (A2), D3.2 (A2), D30.2 (A2), D31.2 (A2), D32.2 (A2), D33.2 (A2), D34.2 (A2), D35.2 (A2), D36.2 (A2), D37.2 (A2), D38.2 (A2), D39.2 (A2), D4.2 (A2), D40.2 (A2), D41.2 (A2), D42.2 (A2), D43.2 (A2), D44.2 (A2), D45.2 (A2), D46.2 (A2), D47.2 (A2), D48.2 (A2), D49.2 (A2), D5.2 (A2), D50.2 (A2), D51.2 (A2), D52.2 (A2), D53.2 (A2), D54.2 (A2), D55.2 (A2), D56.2 (A2), D57.2 (A2), D58.2 (A2), D59.2 (A2), D6.2 (A2), D60.2 (A2), D61.2 (A2), D62.2 (A2), D63.2 (A2), D64.2 (A2), D7.2 (A2), D8.2 (A2), D9.2 (A2), U11.12 (GND), U11.21 (A0), U11.3 (A2), U12.12 (GND), U12.3 (A2), U13.12 (GND), U13.2 (A1), U13.21 (A0)
- net SCL: now also U11.22 (SCL), U12.22 (SCL), U13.22 (SCL)
- net SDA: now also U11.23 (SDA), U12.23 (SDA), U13.23 (SDA)
- net VCC: now also R100.1, R103.1, R104.1, R107.1, R108.1, R111.1, R112.1, R115.1, R116.1, R119.1, R120.1, R123.1, R124.1, R127.1, R128.1, R165.1, R166.1, R167.1, R168.1, R173.1, R174.1, R175.1, R176.1, R181.1, R182.1, R183.1, R184.1, R189.1, R190.1, R191.1, R192.1, R197.1, R198.1, R199.1, R200.1, R205.1, R206.1, R207.1, R208.1, R213.1, R214.1, R215.1, R216.1, R221.1, R222.1, R223.1, R224.1, R67.1, R68.1, R69.1, R70.1, R71.1, R72.1, R73.1, R74.1, R83.1, R85.1, R87.1, R89.1, R91.1, R93.1, R95.1, R97.1, R99.1, U11.24 (VCC), U12.24 (VCC), U13.24 (VCC)
- net VREF_HIGH: now also U11.2 (A1), U12.2 (A1), U12.21 (A0), U13.3 (A2)
- net at U23.4 (P00): now also C13.1, R67.2, R75.2; no longer J103.1 (Pin_1)
- net at U23.14 (P11): now also C30.1, R95.2, R96.2; no longer J103.10 (Pin_10)
- net at U23.15 (P12): now also C29.1, R93.2, R94.2; no longer J103.11 (Pin_11)
- net at J103.12 (Pin_12): now also D13.1 (A1), R92.1; no longer U23.16 (P13)
- net at U23.17 (P14): now also C27.1, R89.2, R90.2; no longer J103.13 (Pin_13)
- net at U23.18 (P15): now also C26.1, R87.2, R88.2; no longer J103.14 (Pin_14)
- net at J103.15 (Pin_15): now also D10.1 (A1), R86.1; no longer U23.19 (P16)
- net at U23.20 (P17): now also C24.1, R83.2, R84.2; no longer J103.16 (Pin_16)
- net at J103.2 (Pin_2): now also D2.1 (A1), R76.1; no longer U23.5 (P01)
- net at J103.3 (Pin_3): now also D3.1 (A1), R77.1; no longer U23.6 (P02)
- net at J103.4 (Pin_4): now also D4.1 (A1), R78.1; no longer U23.7 (P03)
- net at U23.8 (P04): now also C17.1, R71.2, R79.2; no longer J103.5 (Pin_5)
- net at U23.9 (P05): now also C18.1, R72.2, R80.2; no longer J103.6 (Pin_6)
- net at U23.10 (P06): now also C19.1, R73.2, R81.2; no longer J103.7 (Pin_7)
- net at U23.11 (P07): now also C23.1, R74.2, R82.2; no longer J103.8 (Pin_8)
- net at J103.9 (Pin_9): now also D16.1 (A1), R98.1; no longer U23.13 (P10)
- net at U23.1 (~{INT}): now also TP21.1
- new net: C78.1, R223.2, R227.2, U13.11 (P07)
- new net: D27.1 (A1), J46.6 (Pin_6), R121.1
- new net: C42.1, R119.2, R121.2, U11.9 (P05)
- new net: C36.1, R107.2, R109.2, U11.6 (P02)
- new net: D59.1 (A1), J48.7 (Pin_7), R219.1
- new net: D62.1 (A1), J47.9 (Pin_9), R226.1
- new net: C77.1, R222.2, R226.2, U12.13 (P10)
- new net: D38.1 (A1), J47.15 (Pin_15), R178.1
- new net: C53.1, R174.2, R178.2, U12.19 (P16)
- new net: C72.1, R213.2, R217.2, U12.10 (P06)
- new net: D56.1 (A1), J48.11 (Pin_11), R212.1
- new net: C25.1, R85.2, R86.2, U23.19 (P16)
- new net: D17.1 (A1), J46.1 (Pin_1), R101.1
- new net: D30.1 (A1), J46.10 (Pin_10), R126.1
- new net: D28.1 (A1), J46.11 (Pin_11), R122.1
- new net: D26.1 (A1), J46.12 (Pin_12), R118.1
- new net: D24.1 (A1), J46.13 (Pin_13), R114.1
- new net: D22.1 (A1), J46.14 (Pin_14), R110.1
- new net: D20.1 (A1), J46.15 (Pin_15), R106.1
- new net: D18.1 (A1), J46.16 (Pin_16), R102.1
- new net: D19.1 (A1), J46.2 (Pin_2), R105.1
- new net: D21.1 (A1), J46.3 (Pin_3), R109.1
- new net: D23.1 (A1), J46.4 (Pin_4), R113.1
- new net: D25.1 (A1), J46.5 (Pin_5), R117.1
- new net: D29.1 (A1), J46.7 (Pin_7), R125.1
- new net: D31.1 (A1), J46.8 (Pin_8), R129.1
- new net: D32.1 (A1), J46.9 (Pin_9), R163.1
- new net: C64.1, R197.2, R201.2, U12.8 (P04)
- new net: C16.1, R70.2, R78.2, U23.7 (P03)
- new net: C74.1, R215.2, R219.2, U13.10 (P06)
- new net: C47.1, R128.2, R163.2, U11.13 (P10)
- new net: C40.1, R115.2, R117.2, U11.8 (P04)
- new net: C44.1, R123.2, R125.2, U11.10 (P06)
- new net: D45.1 (A1), J47.4 (Pin_4), R193.1
- new net: C60.1, R189.2, R193.2, U12.7 (P03)
- new net: C33.1, R100.2, R102.2, U11.20 (P17)
- new net: C50.1, R167.2, R171.2, U13.4 (P00)
- new net: C71.1, R208.2, R212.2, U13.15 (P12)
- new net: C69.1, R206.2, R210.2, U12.15 (P12)
- new net: C67.1, R200.2, R204.2, U13.16 (P13)
- new net: C79.1, R224.2, R228.2, U13.13 (P10)
- new net: D14.1 (A1), J103.11 (Pin_11), R94.1
- new net: C66.1, R199.2, R203.2, U13.8 (P04)
- new net: C28.1, R91.2, R92.2, U23.16 (P13)
- new net: D55.1 (A1), J48.6 (Pin_6), R211.1
- new net: C35.1, R104.2, R106.2, U11.19 (P16)
- new net: D1.1 (A1), J103.1 (Pin_1), R75.1
- new net: D43.1 (A1), J48.3 (Pin_3), R187.1
- new net: D48.1 (A1), J48.13 (Pin_13), R196.1
- new net: C59.1, R184.2, R188.2, U13.18 (P15)
- new net: C43.1, R120.2, R122.2, U11.15 (P12)
- new net: C55.1, R176.2, R180.2, U13.19 (P16)
- new net: D54.1 (A1), J47.11 (Pin_11), R210.1
- new net: C46.1, R127.2, R129.2, U11.11 (P07)
- new net: C68.1, R205.2, R209.2, U12.9 (P05)
- new net: D11.1 (A1), J103.14 (Pin_14), R88.1
- new net: D39.1 (A1), J48.2 (Pin_2), R179.1
- new net: C32.1, R101.2, R99.2, U11.4 (P00)
- new net: D44.1 (A1), J48.14 (Pin_14), R188.1
- new net: C15.1, R69.2, R77.2, U23.6 (P02)
- new net: D41.1 (A1), J47.3 (Pin_3), R185.1
- new net: C57.1, R182.2, R186.2, U12.18 (P15)
- new net: D60.1 (A1), J48.10 (Pin_10), R220.1
- new net: D33.1 (A1), J47.1 (Pin_1), R169.1
- new net: C48.1, R165.2, R169.2, U12.4 (P00)
- new net: C73.1, R214.2, R218.2, U12.14 (P11)
- new net: D49.1 (A1), J47.5 (Pin_5), R201.1
- new net: C51.1, R168.2, R172.2, U13.20 (P17)
- new net: D5.1 (A1), J103.5 (Pin_5), R79.1
- new net: C39.1, R112.2, R114.2, U11.17 (P14)
- new net: D36.1 (A1), J48.16 (Pin_16), R172.1
- new net: D7.1 (A1), J103.7 (Pin_7), R81.1
- new net: C38.1, R111.2, R113.2, U11.7 (P03)
- new net: D34.1 (A1), J47.16 (Pin_16), R170.1
- new net: C49.1, R166.2, R170.2, U12.20 (P17)
- new net: C75.1, R216.2, R220.2, U13.14 (P11)
- new net: D9.1 (A1), J103.16 (Pin_16), R84.1
- new net: C56.1, R181.2, R185.2, U12.6 (P02)
- new net: TP23.1, U12.1 (~{INT})
- new net: C76.1, R221.2, R225.2, U12.11 (P07)
- new net: C65.1, R198.2, R202.2, U12.16 (P13)
- new net: C61.1, R190.2, R194.2, U12.17 (P14)
- new net: C52.1, R173.2, R177.2, U12.5 (P01)
- new net: D64.1 (A1), J48.9 (Pin_9), R228.1
- new net: D37.1 (A1), J47.2 (Pin_2), R177.1
- new net: C70.1, R207.2, R211.2, U13.9 (P05)
- new net: C41.1, R116.2, R118.2, U11.16 (P13)
- new net: C54.1, R175.2, R179.2, U13.5 (P01)
- new net: C62.1, R191.2, R195.2, U13.7 (P03)
- new net: D35.1 (A1), J48.1 (Pin_1), R171.1
- new net: D53.1 (A1), J47.6 (Pin_6), R209.1
- new net: D50.1 (A1), J47.12 (Pin_12), R202.1
- new net: TP24.1, U13.1 (~{INT})
- new net: C63.1, R192.2, R196.2, U13.17 (P14)
- new net: C58.1, R183.2, R187.2, U13.6 (P02)
- new net: D57.1 (A1), J47.7 (Pin_7), R217.1
- new net: D47.1 (A1), J48.4 (Pin_4), R195.1
- new net: C31.1, R97.2, R98.2, U23.13 (P10)
- new net: D8.1 (A1), J103.8 (Pin_8), R82.1
- new net: D61.1 (A1), J47.8 (Pin_8), R225.1
- new net: D58.1 (A1), J47.10 (Pin_10), R218.1
- new net: D51.1 (A1), J48.5 (Pin_5), R203.1
- new net: C45.1, R124.2, R126.2, U11.14 (P11)
- new net: D52.1 (A1), J48.12 (Pin_12), R204.1
- new net: D40.1 (A1), J48.15 (Pin_15), R180.1
- new net: D63.1 (A1), J48.8 (Pin_8), R227.1
- new net: C14.1, R68.2, R76.2, U23.5 (P01)
- new net: D6.1 (A1), J103.6 (Pin_6), R80.1
- new net: D42.1 (A1), J47.14 (Pin_14), R186.1
- new net: C37.1, R108.2, R110.2, U11.18 (P15)
- new net: D15.1 (A1), J103.10 (Pin_10), R96.1
- new net: D12.1 (A1), J103.13 (Pin_13), R90.1
- new net: D46.1 (A1), J47.13 (Pin_13), R194.1
- new net: C34.1, R103.2, R105.2, U11.5 (P01)
- new net: TP22.1, U11.1 (~{INT})
Other:
- moved on the sheet: J103, U23
