File: New Panel/Main Board/Main Board.kicad_pcb (KiCad board)
At the start: 2 copper layers, 243.2 x 134 mm, 530 parts, among them J10 Conn_02x07_Odd_Even, J102 Speaker Out, J103 Conn_02x08_Odd_Even, J11 Conn_02x07_Odd_Even, J110 SD Holder MEM2061-01-188-00-A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, J12 Conn_02x07_Odd_Even, J13 Conn_01x03_Pin, J14 Conn_01x03_Pin, J15 Conn_01x03_Pin, J16 Conn_01x03_Pin, J17 Conn_01x03_Pin, J18 Conn_01x03_Pin, J19 Conn_01x03_Pin, J2 I2C_MAIN, J20 Conn_01x03_Pin, J21 Conn_01x03_Pin, J22 Conn_01x03_Pin, J23 Conn_01x03_Pin, J24 Conn_01x03_Pin, J25 Conn_01x03_Pin, J26 Conn_01x03_Pin, J27 Conn_01x03_Pin, J28 Conn_01x03_Pin, J29 Conn_01x03_Pin, J3 I2C_A, J30 Conn_01x03_Pin, J31 Conn_01x03_Pin, J32 Conn_01x03_Pin, J33 Conn_01x03_Pin, J34 Conn_01x03_Pin, J35 Conn_01x03_Pin, J36 Conn_01x03_Pin, J37 Conn_01x03_Pin, J38 Conn_01x03_Pin, J39 Conn_01x03_Pin, J4 I2C_B, J40 Conn_01x03_Pin, J41 Conn_01x03_Pin, J42 Conn_01x03_Pin, J43 Conn_01x03_Pin, J44 Conn_01x03_Pin, J45 VCC Select, J46 Conn_02x08_Odd_Even, J47 Conn_02x08_Odd_Even, J48 Conn_02x08_Odd_Even, J5 Conn_02x07_Odd_Even, J6 Conn_02x07_Odd_Even, J7 Conn_02x07_Odd_Even, J8 Conn_02x07_Odd_Even, J85 I2C_C, J86 I2C_D, J87 I2C_E, J88 Neopixel Header, J89 Servo Header B, J9 Conn_02x07_Odd_Even, J90 Servo Header A, J91 Servo Header C, J92 Servo Header D, J93 I2C_F, J94 I2C_G, J95 I2C_H, J96 UART_EXT, J97 Display 1, J98 Display 2, J99 5 VIN, Q1 BSS138, Q2 NPN transistor, SW1 SW_Push, SW2 SW_Push, U1 ESP32-S3-WROOM-1-N4, U10 Analog_MUX_CD4067BPWR, U11 IO_EXPANDER_TCA9535PWR, U12 IO_EXPANDER_TCA9535PWR, U13 IO_EXPANDER_TCA9535PWR, U19 Shift Register SN74HCS164PWR, U2 Analog_MUX_CD4067BPWR, U21 I2C_MUX_TCA9548APWR, U22 Ethernet Adapter, U23 IO_EXPANDER_TCA9535PWR, U3 Analog_MUX_CD4067BPWR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

Commit message: Continued PCB Layout
Parts:
- moved U23 346.2 mm to (190.9, 70.5)
- moved U13 346.1 mm to (180.1, 70.5)
- moved U12 346.0 mm to (169.4, 70.5)
- moved U11 345.9 mm to (158.4, 70.5)
- moved R158 341.0 mm to (160.7, 62.2), turned to -90 degrees
- moved TP24 328.1 mm to (177.2, 61.0)
- moved TP23 325.0 mm to (166.4, 61.0)
- moved R74 322.6 mm to (201.1, 77.5)
- moved TP22 322.3 mm to (155.6, 61.0)
- moved R89 322.2 mm to (193.7, 80.6)
- moved R213 321.2 mm to (185.9, 77.5)
- moved R115 320.7 mm to (155.7, 77.5)
- moved R214 320.5 mm to (185.9, 80.6)
- moved R116 320.0 mm to (155.7, 80.6)
- moved R215 319.8 mm to (185.9, 83.8)
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Connections:
- U10 pad 16: unconnected-(U10-CHANNELIN/OUT15-Pad16) -> /Analog Input Mux/SW15_1
- U10 pad 17: unconnected-(U10-CHANNELIN/OUT14-Pad17) -> /Analog Input Mux/SW14_1
- U10 pad 18: unconnected-(U10-CHANNELIN/OUT13-Pad18) -> /Analog Input Mux/SW13_1
- U10 pad 19: unconnected-(U10-CHANNELIN/OUT12-Pad19) -> /Analog Input Mux/SW12_1
- U10 pad 2: unconnected-(U10-CHANNELIN/OUT7-Pad2) -> /Analog Input Mux/SW7_1
- U10 pad 20: unconnected-(U10-CHANNELIN/OUT11-Pad20) -> /Analog Input Mux/SW11_1
- U10 pad 21: unconnected-(U10-CHANNELIN/OUT10-Pad21) -> /Analog Input Mux/SW10_1
- U10 pad 22: unconnected-(U10-CHANNELIN/OUT9-Pad22) -> /Analog Input Mux/SW9_1
- U10 pad 23: unconnected-(U10-CHANNELIN/OUT8-Pad23) -> /Analog Input Mux/SW8_1
- U10 pad 3: unconnected-(U10-CHANNELIN/OUT6-Pad3) -> /Analog Input Mux/SW6_1
- U10 pad 4: unconnected-(U10-CHANNELIN/OUT5-Pad4) -> /Analog Input Mux/SW5_1
- U10 pad 5: unconnected-(U10-CHANNELIN/OUT4-Pad5) -> /Analog Input Mux/SW4_1
- U10 pad 6: unconnected-(U10-CHANNELIN/OUT3-Pad6) -> /Analog Input Mux/SW3_1
- U10 pad 7: unconnected-(U10-CHANNELIN/OUT2-Pad7) -> /Analog Input Mux/SW2_1
- U10 pad 8: unconnected-(U10-CHANNELIN/OUT1-Pad8) -> /Analog Input Mux/SW1_1
- U10 pad 9: unconnected-(U10-CHANNELIN/OUT0-Pad9) -> /Analog Input Mux/SW0_1
Routing:
- net +12V: track 0.00 -> 220.5 mm
- net +5V_NEOPIXEL: track 0.00 -> 201.5 mm, vias 0 -> 1
- net /Analog Input Mux/Analog_COM: track 0.00 -> 130.5 mm, vias 0 -> 2
- net Net-(J12-Pin_4): track 0.00 -> 89.8 mm, vias 0 -> 1
- net Net-(J12-Pin_2): track 0.00 -> 84.6 mm, vias 0 -> 1
- net Net-(J12-Pin_3): track 0.00 -> 84.3 mm, vias 0 -> 1
- net Net-(J12-Pin_1): track 0.00 -> 79.7 mm, vias 0 -> 1
- net Net-(D17-A1): track 0.00 -> 75.2 mm
- net Net-(J12-Pin_13): track 0.00 -> 72.4 mm, vias 0 -> 1
- net Net-(J12-Pin_11): track 0.00 -> 71.0 mm, vias 0 -> 1
- net Net-(J12-Pin_9): track 0.00 -> 69.7 mm, vias 0 -> 1
- net Net-(J12-Pin_14): track 0.00 -> 68.6 mm, vias 0 -> 1
- net Net-(J12-Pin_12): track 0.00 -> 67.2 mm, vias 0 -> 1
- net Net-(J12-Pin_10): track 0.00 -> 65.9 mm, vias 0 -> 1
- net Net-(J12-Pin_5): track 0.00 -> 65.7 mm, vias 0 -> 1
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- added copper zone on In2.Cu, net +3.3V
- added copper zone on B.Cu, net GND
- added copper zone on F.Cu, net GND
- added copper zone on In1.Cu, net GND
Other:
- copper layers 2 -> 4
