File: New Panel/Main Board/Main Board.kicad_sch (KiCad schematic)
At the start: 80 parts, among them J100 5 VIN alt, J101 VCC Select, J102 Speaker Out, J110 SD Holder MEM2061-01-188-00-A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, J2 I2C_MAIN, J3 I2C_A, J4 I2C_B, J85 I2C_C, J86 I2C_D, J87 I2C_E, J88 Neopixel Header, J89 Servo Header B, J90 Servo Header A, J91 Servo Header C, J92 Servo Header D, J93 I2C_F, J94 I2C_G, J95 I2C_H, J96 UART_EXT, J97 Display 1, J98 Display 2, J99 5 VIN, Q1 BSS138, SW1 SW_Push, SW2 SW_Push, U1 ESP32-S3-WROOM-1-N4, U19 Shift Register SN74HCS164PWR, U20 3v3 Reg AZ1084CD-3.3TRG1, U21 I2C_MUX_TCA9548APWR, U22 Ethernet Adapter

Commit message: adjusted schematic and started PCB Work
Parts:
- removed C23, C24: 5V Line Smoother, Capacitor_THT:CP_Radial_D10.0mm_P2.50mm_P5.00mm, symbol Device:C_Polarized
- removed C25, C26: 3V3 Line Smoother, Capacitor_THT:CP_Radial_D10.0mm_P2.50mm_P5.00mm, symbol Device:C_Polarized
- removed J100: 5 VIN alt, Connector_BarrelJack:BarrelJack_Horizontal, symbol main-eagle-import:DCJ0303
- removed J101: VCC Select, Connector_PinHeader_2.54mm:PinHeader_1x03_P2.54mm_Vertical, symbol Connector:Conn_01x03_Pin
- removed U20: 3v3 Reg AZ1084CD-3.3TRG1, New Panel Parts:TO-252-3_6P6X6P1_DIO, symbol New_Panel_Parts:3v3 Reg AZ1084CD-3.3TRG1
- added C12: 22uF, Capacitor_SMD:C_0603_1608Metric_Pad1.08x0.95mm_HandSolder, symbol Device:C
- added D97, D98, D99: LED, LED_THT:LED_D5.0mm, symbol Device:LED
- added F1: Blade Fuse, New Panel Parts:FUSE_3568, symbol New_Panel_Parts:Blade Fuse Holder 3568
- added J45: VCC Select, Connector_PinHeader_2.54mm:PinHeader_1x02_P2.54mm_Vertical, symbol Connector:Conn_01x02_Pin
- added PS1, PS3: R-78K5.0-2.0, New Panel Parts:CONV_R-78K5.0-2.0, symbol New_Panel_Parts:R-78K5.0-2.0
- added PS2: R-78K3.3-2.0, New Panel Parts:CONV_R-78K3.3-2.0, symbol New_Panel_Parts:R-78K3.3-2.0
- added Q2: NPN transistor, Package_TO_SOT_THT:TO-92_Inline, symbol Transistor_BJT:2N3904
- added R164, R229: 300R, Resistor_SMD:R_0603_1608Metric, symbol Device:R
- added R230: 150, Resistor_SMD:R_0603_1608Metric, symbol Device:R
- added R66: 10K, Resistor_SMD:R_0603_1608Metric, symbol Device:R
- added TP10, TP11, TP12, TP13, TP14, TP15, TP16, TP17, TP18, TP19, TP20, TP9: TestPoint, Connector_Pin:Pin_D1.0mm_L10.0mm, symbol Connector:TestPoint
- C1: value 10uF -> 22uF
- R159, R160, R161, R162: value 10K -> 100K
- U1: footprint SMD -> ESP32 S3:ESP32S3WROOM1N8R2
Connections:
- net +3.3V: now also J45.2 (Pin_2), PS2.3 (+VOUT), R230.1
- net GND: now also C1.2, J89.1 (Pin_1), J90.1 (Pin_1), J91.1 (Pin_1), J92.1 (Pin_1), C12.2, D97.1 (K), D98.1 (K), D99.1 (K), PS1.2 (GND), PS2.2 (GND), PS3.2 (GND), Q2.3 (C); no longer C1.1, J102.2 (Pin_2), J89.3 (Pin_3), J90.3 (Pin_3), J91.3 (Pin_3), J92.3 (Pin_3)
- net Speaker_Out: now also R66.2; no longer J102.1 (Pin_1)
- net at J1.VCC: now also J45.1 (Pin_1)
- net at U1.13 (IO19): now also J91.3 (Pin_3); no longer J91.2 (Pin_2)
- net at U1.14 (IO20): now also J92.3 (Pin_3); no longer J92.2 (Pin_2)
- net at U1.16 (IO46): now also TP14.1
- net at U1.26 (IO45): now also TP13.1
- net at U1.28 (IO35): now also TP9.1
- net at U1.29 (IO36): now also TP10.1
- net at U1.30 (IO37): now also TP11.1
- net at U1.31 (IO38): now also J90.3 (Pin_3); no longer J90.2 (Pin_2)
- net at U1.32 (IO39): now also J89.3 (Pin_3); no longer J89.2 (Pin_2)
- net at U1.35 (IO42): now also TP12.1
- net at U22.5V: now also TP19.1
- net at U22.INT: now also TP20.1
- net at J110.1 (DAT2): now also TP16.1
- net at J110.10 (CD2): now also TP18.1
- net at J110.8 (DAT1): now also TP15.1
- net at J110.9 (CD1): now also TP17.1
- removed net +5V: C1.2, J88.1 (Pin_1), J88.2 (Pin_2), J89.1 (Pin_1), J90.1 (Pin_1), J91.1 (Pin_1), J92.1 (Pin_1), J99.1, R134.1
- new net: D97.2 (A), R164.2
- new net: J102.1 (Pin_1), Q2.1 (E)
- new net: D98.2 (A), R229.2
- new net: F1.1, F1.3, J99.1
- new net: D99.2 (A), R230.2
- new net: Q2.2 (B), R66.1
- new net +12V: F1.2, F1.4, PS1.1 (+VIN), PS2.1 (+VIN), PS3.1 (+VIN)
- new net +5V_NEOPIXEL: C12.1, J102.2 (Pin_2), J88.1 (Pin_1), J88.2 (Pin_2), PS3.3 (+VOUT), R134.1, R164.1
- new net +5V_SERVO: C1.1, J89.2 (Pin_2), J90.2 (Pin_2), J91.2 (Pin_2), J92.2 (Pin_2), PS1.3 (+VOUT), R229.1
Other:
- note removed: "Power Distribution"
- moved on the sheet: J102, J91, J92, J99
